Commit message: add gazebo_plugins and gazebo diff drive

File: robot_pkg/urdf/robot/actuator/caster.urdf.xacro (robot description, xacro)
@@ -29,4 +29,12 @@
             <origin xyz="${xyz_offset}" rpy="0.0 0.0 0.0"/>
         </joint>
+        <gazebo reference="${caster_name}_link">
+            <!-- mu1 切向摩擦，mu2 法向摩擦 kp 刚度 kd 阻尼 -->
+            <mu1 value="0.0"/>
+            <mu2 value="0.0"/>
+            <kp value="1000000000.0"/>
+            <kd value="1.0"/>
+            <material>Gazebo/Black</material>
+        </gazebo>
     </xacro:macro>
 </robot>

File: robot_pkg/urdf/robot/actuator/wheel.urdf.xacro (robot description, xacro)
@@ -30,4 +30,12 @@
             <axis xyz="0 1 0"/>
         </joint>
+        <!-- 添加gazebo插件 -->
+        <gazebo reference="${wheel_name}_link">
+            <mu1 value="20.0"/>
+            <mu2 value="20.0"/>
+            <kp value="1000000000.0"/>
+            <kd value="1.0"/>
+            <material>Gazebo/Yellow</material>
+        </gazebo>
     </xacro:macro>
 </robot>

File: robot_pkg/urdf/robot/robot.urdf.xacro (robot description, xacro)
@@ -7,4 +7,5 @@
     <xacro:include filename="$(find robot_pkg)/urdf/robot/actuator/wheel.urdf.xacro" />
     <xacro:include filename="$(find robot_pkg)/urdf/robot/actuator/caster.urdf.xacro" />
+    <xacro:include filename="$(find robot_pkg)/urdf/robot/plugins/gazebo_control.xacro" />
     <xacro:base_link length="0.1" radius="0.05" />
     <xacro:imu_link imu_name="imu" xyz_offset="0 0 0" />
@@ -15,3 +16,4 @@
     <xacro:caster_link caster_name="front_caster" xyz_offset="0.04 0.0 -0.066" />
     <xacro:caster_link caster_name="back_caster" xyz_offset="-0.04 0.0 -0.066" />
+    <xacro:gazebo_control_plugin separation="0.1" diameter="0.064" />
 </robot>
