Commit message: feat(robot): add gazebo sensor plugin and camera optical link
- Include gazebo_sensor_plugins.xacro in robot.urdf.xacro
- Add xacro:gazebo_sensor_plugin macro call
- Define camera_optical_link in camera.urdf.xacro
- Create fixed joint between camera_link and camera_optical_link
- Update camera joint name from base_link_to_camera to camera_joint

File: robot_pkg/urdf/robot/robot.urdf.xacro (robot description, xacro)
@@ -8,4 +8,5 @@
     <xacro:include filename="$(find robot_pkg)/urdf/robot/actuator/caster.urdf.xacro" />
     <xacro:include filename="$(find robot_pkg)/urdf/robot/plugins/gazebo_control.xacro" />
+    <xacro:include filename="$(find robot_pkg)/urdf/robot/plugins/gazebo_sensor_plugins.xacro" />
     <xacro:base_link length="0.1" radius="0.05" />
     <xacro:imu_link imu_name="imu" xyz_offset="0 0 0" />
@@ -17,3 +18,4 @@
     <xacro:caster_link caster_name="back_caster" xyz_offset="-0.04 0.0 -0.066" />
     <xacro:gazebo_control_plugin separation="0.1" diameter="0.064" />
+    <xacro:gazebo_sensor_plugin />
 </robot>

File: robot_pkg/urdf/robot/sensor/camera.urdf.xacro (robot description, xacro)
@@ -3,4 +3,6 @@
     <xacro:include filename="$(find robot_pkg)/urdf/robot/sensor/common_inertia.urdf.xacro"/>
     <xacro:macro name="camera_link" params = "xyz_offset">
+        <link name="camera_optical_link">
+        </link>
         <link name="camera_link">
             <visual>
@@ -24,9 +26,14 @@
             <xacro:box_inertia m="0.1" w="0.02" h="0.1" d="0.02" />
         </link>
-        <joint name="base_link_to_camera" type="fixed">
+        <joint name="camera_joint" type="fixed">
             <parent link="base_link"/>
             <child link="camera_link"/>
             <origin xyz="${xyz_offset}" rpy="0.0 0.0 0.0"/>
         </joint>
+        <joint name="camera_optical_joint" type="fixed">
+            <parent link="camera_link"/>
+            <child link="camera_optical_link"/>
+            <origin xyz="${xyz_offset}" rpy="${-pi/2} 0.0 ${-pi/2}"/>
+        </joint>
     </xacro:macro>
 </robot>
